File: pcb/kicad/proyek/hgd-v1.kicad_sch (KiCad schematic)
At the start: 12 parts, among them J1 HX711 01x04_Socket, J2 LCD I2C 01x04_Socket, J3 LV Conn_01x06_Socket, J4 HV Conn_01x06_Socket, SW1 SW_Push, U2 ESP32-DEVKIT-V1

Commit message: PCB hgd-v1: log kerja KiCad (langkah 1-3) dan skema terbaru
Co-Authored-By: Claude Opus 5.5 <noreply@anthropic.com>
Claude-Session: https://claude.ai/code/session_015Z5tJC56ToSqz8r7EkyAzt
Parts:
- added D2: RED LED, LED_THT:LED_D3.0mm, symbol Device:LED
- added R2: 220 Ω, Resistor_THT:R_Axial_DIN0207_L6.3mm_D2.5mm_P10.16mm_Horizontal, symbol Device:R
Connections:
- net GND: now also D2.1 (K)
- net at C1.1, C2.1, J1.4 (VCC)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: now also R2.1
- new net: D2.2 (A), R2.2
- no-connect marks 0 -> 24
Other:
- note added: "3mm"
- note added: "5mm"
- company: (none) -> Kelompok 01
- title: (none) -> Hand Grip Dynamometer

Commit message: PCB: versi akhir 26 Okt. 2026 (skema, papan, PDF skema, tangkapan)
- hgd-v1.kicad_sch: judul "Digital Hand Grip Dynamometer" (hanya title block).
- hgd-v1.kicad_pcb: jalur ulang dengan posisi footprint tetap (56 via GND),
  silkscreen tiga baris, stackup FR4 1,6 mm; folder keluaran Gerber kembali
  ke gerber/ (tanpa jalur lokal).
- hgd-v1.kicad_pro baru (jalur keluaran relatif di dalam proyek).
- PDF skema, tangkapan Assign Footprints, ERC, DRC, dan render papan/3D.
- Desain PCB v8 (Bagian 8.1a daftar Assign Footprints), log kerja KiCad v2,
  README KiCad v6, catatan proyek v59.
- Gambar penempatan, salinan verbatim, dan STEP tetap versi 17 Okt.;
  Gerber tetap di luar repo sampai disetujui.

Co-Authored-By: Claude Opus 5.5 <noreply@anthropic.com>
Other:
- title: Hand Grip Dynamometer -> Digital Hand Grip Dynamometer
Changed lines of the file:
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@@
 	(paper "A4")
 	(title_block
-		(title "Hand Grip Dynamometer")
-		(date "2026-10-17")
+		(title "Digital Hand Grip Dynamometer")
+		(date "2026-10-19")
 		(rev "1")
 		(company "Kelompok 01")
